File: hardware/tracker/tracker.sch (EAGLE design)
At the start: 24 parts, among them IC1 TP4056, IC2 LM1117MPX-3.3, SW1 PWR-SWITCH, X1 MINI-USB-SCHIELD-32005-301

Commit message: no message
Connections:
- net N$2: now also U$1.ANODE@1, U$1.ANODE@2; no longer U$1.ANODE$1, U$1.ANODE$2
- net N$3: now also U$2.ANODE@1, U$2.ANODE@2; no longer U$2.ANODE$1, U$2.ANODE$2
- net N$4: now also U$3.ANODE@1, U$3.ANODE@2; no longer U$3.ANODE$1, U$3.ANODE$2
- net N$5: now also U$4.ANODE@1, U$4.ANODE@2; no longer U$4.ANODE$1, U$4.ANODE$2
- net N$6: now also U$5.ANODE@1, U$5.ANODE@2; no longer U$5.ANODE$1, U$5.ANODE$2
Changed lines of the file:
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@@
 <net name="N$2" class="0">
 <segment>
-<pinref part="U$1" gate="G$1" pin="ANODE$2"/>
-<pinref part="U$1" gate="G$1" pin="ANODE$1"/>
+<pinref part="U$1" gate="G$1" pin="ANODE@2"/>
+<pinref part="U$1" gate="G$1" pin="ANODE@1"/>
 <wire x1="0" y1="-132.08" x2="0" y2="-129.54" width="0.1524" layer="91"/>
 </segment>
@@
 <net name="N$3" class="0">
 <segment>
-<pinref part="U$2" gate="G$1" pin="ANODE$2"/>
-<pinref part="U$2" gate="G$1" pin="ANODE$1"/>
+<pinref part="U$2" gate="G$1" pin="ANODE@2"/>
+<pinref part="U$2" gate="G$1" pin="ANODE@1"/>
 <wire x1="35.56" y1="-132.08" x2="35.56" y2="-129.54" width="0.1524" layer="91"/>
 </segment>
@@
 <net name="N$4" class="0">
 <segment>
-<pinref part="U$3" gate="G$1" pin="ANODE$2"/>
-<pinref part="U$3" gate="G$1" pin="ANODE$1"/>
+<pinref part="U$3" gate="G$1" pin="ANODE@2"/>
+<pinref part="U$3" gate="G$1" pin="ANODE@1"/>
 <wire x1="71.12" y1="-132.08" x2="71.12" y2="-129.54" width="0.1524" layer="91"/>
 </segment>
@@
 <net name="N$5" class="0">
 <segment>
-<pinref part="U$4" gate="G$1" pin="ANODE$2"/>
-<pinref part="U$4" gate="G$1" pin="ANODE$1"/>
+<pinref part="U$4" gate="G$1" pin="ANODE@2"/>
+<pinref part="U$4" gate="G$1" pin="ANODE@1"/>
 <wire x1="106.68" y1="-132.08" x2="106.68" y2="-129.54" width="0.1524" layer="91"/>
 </segment>
@@
 <net name="N$6" class="0">
 <segment>
-<pinref part="U$5" gate="G$1" pin="ANODE$2"/>
-<pinref part="U$5" gate="G$1" pin="ANODE$1"/>
+<pinref part="U$5" gate="G$1" pin="ANODE@2"/>
+<pinref part="U$5" gate="G$1" pin="ANODE@1"/>
 <wire x1="142.24" y1="-132.08" x2="142.24" y2="-129.54" width="0.1524" layer="91"/>
 </segment>

Commit message: no message
Parts:
- removed D2: (no value), diode:DIODE-SOD106-R
- removed IC2: LM1117MPX-3.3, lm1117:LM1117MPX-3.3
- removed U$1, U$2, U$3, U$4, U$5: KCSA02-109-SMALL, kcsx02:KCSA02-109-SMALL
- removed U$8: FGPMMOPA6C, FGPMMOPA6C:FGPMMOPA6C
- removed U$9: BMP085, bmp085:BMP085
- added C1, C10, C5, C6, C7: (no value), resistor:C-EUC0805K
- added C8: 10uF, resistor:CPOL-EUB/3528-21W
- added JTAG: (no value), PLL:PINHD-1X8
- added LED1: (no value), led:LEDSML1206
- added Q1: IRLML5203, transistor-power:IRLML5203
- added R2: (no value), resistor:R-EU_R0805
- added R3, R4, R5: 10k, resistor:R-EU_R0805
- added U$13: LP2985AIM5-3.3, LP2985:LP2985AIM5-3.3
- C2, C4: device resistor:CPOL-EUB -> resistor:CPOL-EUB/3528-21W
- C3: value 10uF -> (none); device resistor:CPOL-EUB -> resistor:C-EUC0805K
- D1: value (none) -> GF1; device diode:DIODE-SOD106-R -> diode:GF1
- U$11: value CC2540-MINI-BLE -> STM32F103C8; device cc2540:CC2540-MINI-BLE -> stm32:STM32F103C8
Connections:
- removed net A: U$1.A, U$2.A, U$3.A, U$4.A, U$5.A
- removed net B: U$1.B, U$2.B, U$3.B, U$4.B, U$5.B
- removed net C: U$1.C, U$2.C, U$3.C, U$4.C, U$5.C
- removed net D: U$1.D, U$2.D, U$3.D, U$4.D, U$5.D
- removed net E: U$1.E, U$2.E, U$3.E, U$4.E, U$5.E
- removed net F: U$1.F, U$2.F, U$3.F, U$4.F, U$5.F
- removed net G: U$1.G, U$2.G, U$3.G, U$4.G, U$5.G
- removed net H: U$1.DP, U$2.DP, U$3.DP, U$4.DP, U$5.DP
- removed net N$2: U$1.ANODE@1, U$1.ANODE@2
- removed net N$3: U$2.ANODE@1, U$2.ANODE@2
- removed net N$4: U$3.ANODE@1, U$3.ANODE@2
- removed net N$5: U$4.ANODE@1, U$4.ANODE@2
- removed net N$6: U$5.ANODE@1, U$5.ANODE@2
- removed net N$8: IC2.IN, SW1.PWR-OUT1
- new net ADXL_INT1: U$10.INT1
- new net ADXL_INT2: U$10.INT2
- new net BOOT0: U$11.BOOT0
- new net BYPASS: C3.1, U$13.BYPASS
- new net DISPLAY_ON: SW1.BTN2, SW1.PWR-OUT2
- new net EXTERNAL_POWER: R2.2
- new net N$1: Q1.D, SW1.BTN1, SW1.PWR-IN
- new net N$13: JTAG.3, U$11.JTCK/SWCLK
- new net N$16: JTAG.4, U$11.JTDI
- new net N$17: JTAG.5, U$11.JTDO
- new net N$18: JTAG.6, U$11.JNTRST
- new net POWER: D1.C, SW1.PWR-OUT1, U$13.ON/OFF, U$13.VIN
- new net RESET: C10.1, JTAG.7, U$11.NRST
- new net SCL: R4.1, U$10.SCLK, U$11.PB6/I2C1_SCL/TIM4_CH1
- new net SDA: R5.1, U$10.MOSI, U$11.PB7/I2C1_SDA/TIM4_CH2
- net +3V3: now also C1.1, C5.1, C6.1, C7.1, C8.+, JTAG.1, R4.2, R5.2, U$10.!CS, U$10.VDDIO, U$10.VS, U$11.AVCC, U$11.VCC@1, U$11.VCC@2, U$11.VCC@3, U$12.VDD, U$13.VOUT; no longer C3.+, IC2.OUT, IC2.OUT1
- net +5V: now also Q1.G, R2.1, R3.2
- net BAT+: now also Q1.S; no longer D2.A
- net GND: now also C1.2, C10.2, C3.2, C5.2, C6.2, C7.2, C8.-, JTAG.8, R3.1, U$10.MISO, U$11.AGND, U$11.GND@1, U$11.GND@2, U$11.GND@3, U$12.GND, U$12.SHIELD@1, U$12.SHIELD@2, U$12.SHIELD@3, U$12.SHIELD@4, U$13.GND; no longer C3.-, IC2.GND, U$11.GND, U$8.GND@1, U$8.GND@2, U$8.GND@3, U$8.GND@4, U$8.GND@5, U$9.GND
- net N$7: now also JTAG.2, U$11.JTMS/SWDIO; no longer D1.C, D2.C, SW1.PWR-IN
Other:
- moved on the sheet: BTN1, BTN2, C4, R1, SW1, U$10

Commit message: Board version 1
Parts:
- added C11, C9: (no value), resistor:C-EUC0805K
- added Q2: (no value), crystal:CRYSTALHC49S
- added R10, R11: 10k, resistor:R-EU_R0805
- added R12: BOOT0, resistor:R-EU_R0805
- added R13: BOOT1, resistor:R-EU_R0805
- added R6, R7: (no value), resistor:R-EU_R0805
- added R8: 22, resistor:R-EU_R0805
- added R9: 330, resistor:R-EU_R0805
- R2: value (none) -> 22
Connections:
- removed net EXTERNAL_POWER: R2.2
- new net BOOT1: R11.1, R13.1, U$11.PB2/BOOT1
- new net BUTTON1: BTN1.2, R6.2, U$11.PB10/I2C2_SCL/USART3_TX
- new net BUTTON2: BTN2.2, R7.2, U$11.PB11/I2C2_SDA/USART3_RX
- new net N$2: C9.1, Q2.1, U$11.OSC_IN
- new net N$3: C11.1, Q2.2, U$11.OSC_OUT
- new net N$4: R2.1, U$11.PA11/USART1_CTS/CANRX/USBDM/TIM1_CH4
- new net N$5: R8.1, U$11.PA12/USART1_RTS/CAN_TX/USBDP/TIM1_ETR
- new net N$6: LED1.A, R9.1
- new net N$8: R9.2, U$11.PC13/TAMPER-RTC
- new net SD-CD: U$12.CD
- new net SD-CS: U$11.PA4/SPI1_NSS/USART2_CK/ADC12_IN4, U$12.CD/DAT3/CS
- new net SD-DI: U$11.PA7/SPI1_MOSI/ADC12_IN7/TIM3_CH2, U$12.CMD/DI
- new net SD-DO: U$11.PA6/SPI1_MISO/ADC12_IN6/TIM3_CH1, U$12.DAT0/DO
- new net SD-SCLK: U$11.PA5/SPI1_SCK/ADC12_IN5, U$12.CLK/SCLK
- net +3V3: now also R10.2, R11.2, R6.1, R7.1
- net +5V: no longer R2.1
- net ADXL_INT1: now also U$11.PB14/SPI2_MISO/USART3_RTS/TIM1_CH2N
- net ADXL_INT2: now also U$11.PB15/SPI2_MOSI/TIM1_CH3N
- net BOOT0: now also R10.1, R12.1
- net CHARGER_CHARGING: now also U$11.PB8/TIM4_CH3
- net CHARGER_ENABLE: now also U$11.PB5/I2C1_SMBAI
- net CHARGER_STANDBY: now also U$11.PB9/TIM4_CH4
- net GND: now also BTN1.1@1, BTN1.1@2, BTN2.1@1, BTN2.1@2, C11.2, C9.2, LED1.C, R12.2, R13.2
- net USB+D: now also R8.2
- net USB-D: now also R2.2
Other:
- moved on the sheet: BTN1, BTN2, R2
