File: hardware/tracker/tracker.brd (EAGLE design)
At the start: 70 x 65 mm, 24 parts, among them IC1 TP4056, IC2 LM1117MPX-3.3, SW1 PWR-SWITCH, X1 MINI-USB-SCHIELD-32005-301

Commit message: no message
Parts:
- removed D2: (no value), diode:SOD106-R
- removed IC2: LM1117MPX-3.3, lm1117:SOT223
- removed U$1, U$2, U$3, U$4, U$5: KCSA02-109-SMALL, kcsx02:KCSX02-SM
- removed U$8: FGPMMOPA6C, FGPMMOPA6C:FGPMMOPA6C
- removed U$9: BMP085, bmp085:BMP085
- added C1, C10, C5, C6, C7: (no value), resistor:C0805K
- added C8: 10uF, resistor:B/3528-21W
- added JTAG: (no value), PLL:PLL1.27-1X8
- added LED1: (no value), led:SML1206
- added Q1: IRLML5203, transistor-power:MICRO3
- added R2: (no value), resistor:R0805
- added R3, R4, R5: 10k, resistor:R0805
- added U$13: LP2985AIM5-3.3, LP2985:SOT25
- C2, C4: device resistor:PANASONIC_B -> resistor:B/3528-21W
- C3: value 10uF -> (none); device resistor:PANASONIC_B -> resistor:C0805K
- D1: value (none) -> GF1; device diode:SOD106-R -> diode:SMA-DO214AC
- U$11: value CC2540-MINI-BLE -> STM32F103C8; device cc2540:CC2540-MINI-BLE -> stm32:LQFP48-7X7
- U$12: device micro-sd:MICROSD -> micro-sd:C12075
- moved R1 57.0 mm to (15.0, 60.0), flipped to the top, turned to 0 degrees
- moved C2 53.9 mm to (30.0, 60.0), turned to 0 degrees
- moved U$11 53.2 mm to (16.0, 40.0), turned to 0 degrees
- moved IC1 49.5 mm to (22.0, 58.0), flipped to the top, turned to 0 degrees
- moved U$12 49.1 mm to (11.5, 22.5), turned to 270 degrees
- moved U$10 43.1 mm to (25.0, 27.0), flipped to the bottom
- moved D1 41.0 mm to (14.8, 55.0)
- moved C3 40.2 mm to (26.9, 51.7), turned to 270 degrees
- moved C4 3.61 mm to (18.0, 6.00), turned to 90 degrees
Connections:
- removed net A: U$1.7, U$2.7, U$3.7, U$4.7, U$5.7
- removed net B: U$1.6, U$2.6, U$3.6, U$4.6, U$5.6
- removed net C: U$1.4, U$2.4, U$3.4, U$4.4, U$5.4
- removed net D: U$1.2, U$2.2, U$3.2, U$4.2, U$5.2
- removed net E: U$1.1, U$2.1, U$3.1, U$4.1, U$5.1
- removed net F: U$1.9, U$2.9, U$3.9, U$4.9, U$5.9
- removed net G: U$1.10, U$2.10, U$3.10, U$4.10, U$5.10
- removed net H: U$1.5, U$2.5, U$3.5, U$4.5, U$5.5
- removed net N$2: U$1.3, U$1.8
- removed net N$3: U$2.3, U$2.8
- removed net N$4: U$3.3, U$3.8
- removed net N$5: U$4.3, U$4.8
- removed net N$6: U$5.3, U$5.8
- removed net N$8: IC2.3, SW1.3
- removed net VBACKUP: U$8.4
- removed net VCC: U$11.3, U$8.1
- removed net VDDA: U$9.3
- removed net VDDD: U$9.4
- removed net VDDIO: U$10.1
- removed net VS: U$10.6
- new net ADXL_INT1: U$10.8
- new net ADXL_INT2: U$10.9
- new net BOOT0: U$11.44
- new net BYPASS: C3.1, U$13.4
- new net DISPLAY_ON: SW1.4, SW1.5
- new net EXTERNAL_POWER: R2.2
- new net N$1: Q1.3, SW1.1, SW1.2
- new net N$13: JTAG.3, U$11.37
- new net N$16: JTAG.4, U$11.38
- new net N$17: JTAG.5, U$11.39
- new net N$18: JTAG.6, U$11.40
- new net POWER: D1.K, SW1.3, U$13.1, U$13.3
- new net RESET: C10.1, JTAG.7, U$11.7
- new net SCL: R4.1, U$10.14, U$11.42
- new net SDA: R5.1, U$10.13, U$11.43
- new net VBAT: U$11.1
- net +3V3: now also C1.1, C5.1, C6.1, C7.1, C8.+, JTAG.1, R4.2, R5.2, U$10.1, U$10.6, U$10.7, U$11.24, U$11.36, U$11.48, U$11.9, U$12.4, U$13.5; no longer C3.+, IC2.2, IC2.TAB
- net +5V: now also Q1.1, R2.1, R3.2
- net BAT+: now also Q1.2; no longer D2.A
- net GND: now also C1.2, C10.2, C3.2, C5.2, C6.2, C7.2, C8.-, JTAG.8, R3.1, U$10.12, U$11.23, U$11.35, U$11.47, U$11.8, U$12.6, U$12.GND@1, U$12.GND@2, U$12.GND@3, U$12.GND@4, U$13.2; no longer C3.-, IC2.1, U$11.2, U$8.11, U$8.12, U$8.13, U$8.3, U$8.8, U$9.1
- net N$7: now also JTAG.2, U$11.34; no longer D1.C, D2.C, SW1.2
Routing:
- net +3V3: track 0.00 -> 12.7 mm
- net GND: track 0.00 -> 10.4 mm
Other:
- board size 70 x 65 mm -> 39 x 65 mm

Commit message: Board version 1
Parts:
- added C11, C9: (no value), resistor:C0805K
- added Q2: (no value), crystal:HC49/S
- added R10, R11: 10k, resistor:R0805
- added R12: BOOT0, resistor:R0805
- added R13: BOOT1, resistor:R0805
- added R6, R7: (no value), resistor:R0805
- added R8: 22, resistor:R0805
- added R9: 330, resistor:R0805
- R2: value (none) -> 22
- moved LED1 64.3 mm to (17.0, 59.0), flipped to the bottom, turned to 270 degrees
- moved R1 49.3 mm to (24.0, 11.5), flipped to the bottom, turned to 180 degrees
- moved IC1 46.1 mm to (25.5, 12.0), turned to 90 degrees
- moved D1 38.2 mm to (24.3, 18.0), turned to 0 degrees
- moved R4 24.0 mm to (26.0, 21.0), flipped to the bottom, turned to 180 degrees
- moved R5 18.0 mm to (26.0, 24.0), flipped to the bottom, turned to 180 degrees
- moved R2 17.3 mm to (2.00, 14.0), flipped to the bottom, turned to 270 degrees
- moved U$10 11.4 mm to (14.0, 24.0), turned to 90 degrees
- moved R3 10.0 mm to (9.60, 48.6), turned to 0 degrees
- moved C3 9.18 mm to (22.4, 59.7), turned to 0 degrees
- moved C8 8.28 mm to (22.5, 52.5), turned to 180 degrees
- moved C4 5.80 mm to (12.2, 6.00)
- moved U$13 5.02 mm to (22.5, 56.6), turned to 90 degrees
- moved C2 3.20 mm to (28.0, 57.5), turned to 90 degrees
- moved Q1 0.71 mm to (9.20, 51.8), turned to 90 degrees
Connections:
- removed net EXTERNAL_POWER: R2.2
- new net BOOT1: R11.1, R13.1, U$11.20
- new net BUTTON1: BTN1.1, R6.2, U$11.21
- new net BUTTON2: BTN2.1, R7.2, U$11.22
- new net N$2: C9.1, Q2.1, U$11.5
- new net N$3: C11.1, Q2.2, U$11.6
- new net N$4: R2.1, U$11.32
- new net N$5: R8.1, U$11.33
- new net N$6: LED1.A, R9.1
- new net N$8: R9.2, U$11.2
- new net SD-CD: U$12.CD
- new net SD-CS: U$11.14, U$12.2
- new net SD-DI: U$11.17, U$12.3
- new net SD-DO: U$11.16, U$12.7
- new net SD-SCLK: U$11.15, U$12.5
- net +3V3: now also R10.2, R11.2, R6.1, R7.1
- net +5V: no longer R2.1
- net ADXL_INT1: now also U$11.27
- net ADXL_INT2: now also U$11.28
- net BOOT0: now also R10.1, R12.1
- net CHARGER_CHARGING: now also U$11.45
- net CHARGER_ENABLE: now also U$11.41
- net CHARGER_STANDBY: now also U$11.46
- net GND: now also BTN1.2, BTN1.3, BTN2.2, BTN2.3, C11.2, C9.2, LED1.C, R12.2, R13.2
- net USB+D: now also R8.2
- net USB-D: now also R2.2
Routing:
- net GND: track 10.4 -> 311.2 mm, vias 0 -> 8
- net +3V3: track 12.7 -> 113.2 mm, vias 0 -> 8
- net +5V: track 0.00 -> 91.3 mm, vias 0 -> 4
- net BAT+: track 0.00 -> 84.1 mm, vias 0 -> 1
- net POWER: track 0.00 -> 79.3 mm, vias 0 -> 5
- net CHARGER_STANDBY: track 0.00 -> 57.5 mm, vias 0 -> 3
- net BUTTON2: track 0.00 -> 52.5 mm, vias 0 -> 2
- net SCL: track 0.00 -> 46.4 mm, vias 0 -> 4
- net CHARGER_CHARGING: track 0.00 -> 43.1 mm, vias 0 -> 5
- net N$18: track 0.00 -> 40.8 mm, vias 0 -> 1
- net BUTTON1: track 0.00 -> 38.3 mm, vias 0 -> 2
- net CHARGER_ENABLE: track 0.00 -> 36.5 mm, vias 0 -> 3
- net BOOT0: track 0.00 -> 35.7 mm, vias 0 -> 4
- net N$5: track 0.00 -> 31.8 mm, vias 0 -> 2
- net N$4: track 0.00 -> 30.6 mm, vias 0 -> 2
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- added copper zone on layer 1, net GND
- added copper zone on layer 16, net GND

Commit message: Rev A board
Parts:
- moved Q2 1.00 mm to (25.0, 43.0)
- moved C11 0.50 mm to (26.0, 37.5)
- turned R9 to 270 degrees
Routing:
- net GND: track 311.2 -> 316.6 mm, vias 8 -> 6
- net N$8: track 17.1 -> 11.9 mm
- net N$6: track 5.60 -> 3.31 mm
- net N$2: track 12.1 -> 10.1 mm
- net BOOT0: track 35.7 -> 36.4 mm
